Commit message: Fix Flask web server path, add battery display, camera link, and supporting files
Fix FLASK_APP path in start_web.launch.py to correctly point to the installed
app.py location. Add battery state subscription to OLED display node, camera
joint to URDF, and various supporting scripts and config files. Add .gitignore
for build artifacts.

Co-Authored-By: Claude Opus 4.6 (1M context) <noreply@anthropic.com>

File: src/krytn/robot_description/krytn.urdf.xacro (robot description, xacro)
@@ -11,4 +11,10 @@
     <origin xyz="0 0 0.15" rpy="0 0 0" />
   </xacro:lidar_2d>
+  <link name="camera" />
+  <joint name="camera_joint">
+    <parent name="base_link" />
+    <child name="camera" />
+    <origin xyz="-0.05 0.05 0.8" rpy="0 0 ${pi/2}" />
+  </joint>
 <!-- ROS 2 Control block -->
   <ros2_control name="ubiquity_motor_ros2/MotorHardware" type="system">
